File: Schematics/Keybed/LT6502_KEYBED.kicad_pcb (KiCad board)
At the start: 4 copper layers, 261 x 130 mm, 169 parts, among them J14 KeyConn, J4 Conn_02x05_Odd_Even, Q3 STL9P3LLH6, SW1 SW_Push, SW10 SW_Push, SW11 SW_Push, SW12 SW_Push, SW13 SW_Push, SW14 SW_Push, SW15 SW_Push, SW16 SW_Push, SW17 SW_Push, SW18 SW_Push, SW19 SW_Push, SW2 SW_Push, SW20 SW_Push, SW21 SW_Push, SW22 SW_Push, SW23 SW_Push, SW24 SW_Push, SW25 SW_Push, SW26 SW_Push, SW27 SW_Push, SW28 SW_Push, SW29 SW_Push, SW3 SW_Push, SW30 SW_Push, SW31 SW_Push, SW32 SW_Push, SW33 SW_Push, SW34 SW_Push, SW35 SW_Push, SW36 SW_Push, SW37 SW_Push, SW38 SW_Push, SW39 SW_Push, SW4 SW_Push, SW40 SW_Push, SW41 SW_Push, SW42 SW_Push, SW43 SW_Push, SW44 SW_Push, SW45 SW_Push, SW46 SW_Push, SW47 SW_Push, SW48 SW_Push, SW49 SW_Push, SW5 SW_Push, SW50 SW_Push, SW51 SW_Push, SW52 SW_Push, SW53 SW_Push, SW54 SW_Push, SW55 SW_Push, SW57 SW_Push, SW58 SW_Push, SW59 SW_Push, SW6 SW_Push, SW60 SW_Push, SW61 SW_Push, SW65 SW_Push, SW7 SW_Push, SW8 SW_Push, SW9 SW_Push, U1 ATmega644P-20P, U2 74HC138, X2 CXO_DIP8

Commit message: Routing Completed
Routing completed, removed silkscreen IDs for clarity
Parts:
- U2: value 74HC138 -> 74HC238
- moved R3 8.94 mm to (213.1, 179.4), turned to 90 degrees
Routing:
- net ROW7: track 63.0 -> 372.7 mm, vias 0 -> 2
- net /KeyMatrix/COL3: track 165.9 -> 469.3 mm, vias 5 -> 10
- net /KeyMatrix/COL2: track 160.1 -> 426.2 mm, vias 6 -> 13
- net KEYLED0: track 0.00 -> 262.8 mm, vias 0 -> 2
- net ROW0: track 0.00 -> 259.9 mm, vias 0 -> 4
- net /KeyMatrix/COL0: track 95.4 -> 345.4 mm, vias 4 -> 11
- net /KeyMatrix/COL1: track 162.1 -> 411.4 mm, vias 5 -> 10
- net ROW2: track 93.3 -> 272.8 mm, vias 0 -> 5
- net /KeyMatrix/COL6: track 216.4 -> 370.0 mm, vias 6 -> 10
- net ROW3: track 127.2 -> 266.5 mm, vias 1 -> 5
- net AVR_TDO: track 0.00 -> 138.9 mm, vias 0 -> 4
- net DISP_A0: track 0.00 -> 96.4 mm, vias 0 -> 2
- net DISP_A1: track 0.00 -> 95.0 mm, vias 0 -> 2
- net DISP_A2: track 0.00 -> 94.1 mm, vias 0 -> 2
- net ROW5: track 268.1 -> 357.3 mm, vias 4 -> 5
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