File: Schematics/Keybed/LT6502_KEYBED.kicad_pcb (KiCad board)
At the start: 4 copper layers, 261 x 130 mm, 169 parts, among them J14 KeyConn, J4 Conn_02x05_Odd_Even, Q3 STL9P3LLH6, SW1 SW_Push, SW10 SW_Push, SW11 SW_Push, SW12 SW_Push, SW13 SW_Push, SW14 SW_Push, SW15 SW_Push, SW16 SW_Push, SW17 SW_Push, SW18 SW_Push, SW19 SW_Push, SW2 SW_Push, SW20 SW_Push, SW21 SW_Push, SW22 SW_Push, SW23 SW_Push, SW24 SW_Push, SW25 SW_Push, SW26 SW_Push, SW27 SW_Push, SW28 SW_Push, SW29 SW_Push, SW3 SW_Push, SW30 SW_Push, SW31 SW_Push, SW32 SW_Push, SW33 SW_Push, SW34 SW_Push, SW35 SW_Push, SW36 SW_Push, SW37 SW_Push, SW38 SW_Push, SW39 SW_Push, SW4 SW_Push, SW40 SW_Push, SW41 SW_Push, SW42 SW_Push, SW43 SW_Push, SW44 SW_Push, SW45 SW_Push, SW46 SW_Push, SW47 SW_Push, SW48 SW_Push, SW49 SW_Push, SW5 SW_Push, SW50 SW_Push, SW51 SW_Push, SW52 SW_Push, SW53 SW_Push, SW54 SW_Push, SW55 SW_Push, SW57 SW_Push, SW58 SW_Push, SW59 SW_Push, SW6 SW_Push, SW60 SW_Push, SW61 SW_Push, SW65 SW_Push, SW7 SW_Push, SW8 SW_Push, SW9 SW_Push, U1 ATmega644P-20P, U2 74HC238, X2 CXO_DIP8

Commit message: edited PCB dimensions
Loved LHS in 0.5mm to ensure it clears the case edge
Other:
- board size 261 x 130 mm -> 260.5 x 130 mm
Changed lines of the file:
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@@
 	)
 	(gr_line
-		(start 197 120)
+		(start 197.5 120)
 		(end 205 120)
 		(stroke
@@
 	(gr_line
 		(start 458 231)
-		(end 197 231)
+		(end 197.5 231)
 		(stroke
 			(width 0.05)
@@
 	)
 	(gr_line
-		(start 197 231)
-		(end 197 120)
+		(start 197.5 231)
+		(end 197.5 120)
 		(stroke
 			(width 0.05)
