File: Schematics/Keybed/LT6502_KEYBED.kicad_pcb (KiCad board)
At the start: 4 copper layers, 260.5 x 130 mm, 169 parts, among them J14 KeyConn, J4 Conn_02x05_Odd_Even, Q3 STL9P3LLH6, SW1 SW_Push, SW10 SW_Push, SW11 SW_Push, SW12 SW_Push, SW13 SW_Push, SW14 SW_Push, SW15 SW_Push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

Commit message: Updated BoMs ordered PCBs
Parts:
- U2: value 74HC238 -> 74HCT138
