File: Schematics/Keybed/keyleds.kicad_sch (KiCad schematic)
At the start: 23 parts

Commit message: Updated BoMs ordered PCBs
Parts:
- D56, D60, D61, D62, D63, D64, D65, D66, D67, D68, D69: LCSC (none) -> C3030991
- JP1: LCSC (none) -> DNF
