File: Schematics/LT6502/Audio.kicad_sch (KiCad schematic)
At the start: 12 parts, among them U11 LM386

Commit message: Updated BoMs ordered PCBs
Parts:
- C45: LCSC (none) -> C21117
- C46: LCSC C49678 -> C113803
- C54: LCSC C49678 -> C15850
- C55: LCSC (none) -> C1622
- C56, LS1, R87, R88, U11: LCSC (none) -> DNF; now not fitted
- R85: LCSC C23179 -> C25744
- R86: LCSC (none) -> C844598
- VR1: LCSC DNP -> DNF; now not fitted
Changed lines of the file:
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@@
 		(in_bom yes)
 		(on_board yes)
-		(dnp no)
+		(dnp yes)
 		(fields_autoplaced yes)
 		(property "Reference" "C56"
@@
 			)
 		)
+		(property "LCSC" "DNF"
+			(at 222.25 76.2 90)
+			(effects
+				(font
+					(size 1.27 1.27)
+				)
+				(hide yes)
+			)
+		)
 		(pin "1"
 		)
@@
 			)
 		)
-		(property "LCSC" ""
+		(property "LCSC" "C21117"
 			(at 163.83 85.09 0)
 			(effects
@@
 		(in_bom yes)
 		(on_board yes)
-		(dnp no)
+		(dnp yes)
 		(property "Reference" "VR1"
 			(at 101.6 123.19 0)
@@
 			)
 		)
-		(property "LCSC" "DNP"
+		(property "LCSC" "DNF"
 			(at 88.9 115.57 0)
 			(effects
@@
 		(in_bom yes)
 		(on_board yes)
-		(dnp no)
+		(dnp yes)
 		(property "Reference" "R87"
 			(at 82.5712 87.9679 90)
@@
 			)
 		)
-		(property "LCSC" ""
+		(property "LCSC" "DNF"
 			(at 82.55 92.71 90)
 			(effects
@@
 		(in_bom yes)
 		(on_board yes)
-		(dnp no)
+		(dnp yes)
 		(property "Reference" "R88"
 			(at 53.6779 99.0388 90)
@@
 			)
 		)
-		(property "LCSC" ""
+		(property "LCSC" "DNF"
 			(at 58.42 99.06 90)
 			(effects
@@
 			)
 		)
-		(property "LCSC" "C23179"
+		(property "LCSC" "C25744"
 			(at 152.4 91.44 90)
 			(effects
@@
 			)
 		)
-		(property "LCSC" "C49678"
+		(property "LCSC" "C15850"
 			(at 157.48 57.15 0)
 			(effects
@@
 		(in_bom yes)
 		(on_board yes)
-		(dnp no)
+		(dnp yes)
 		(fields_autoplaced yes)
 		(property "Reference" "LS1"
@@
 				)
 				(justify left top)
+				(hide yes)
+			)
+		)
+		(property "LCSC" "DNF"
+			(at 237.49 76.2 0)
+			(effects
+				(font
+					(size 1.27 1.27)
+				)
 				(hide yes)
 			)
@@
 			)
 		)
+		(property "LCSC" "C844598"
+			(at 187.96 99.06 0)
+			(effects
+				(font
+					(size 1.27 1.27)
+				)
+				(hide yes)
+			)
+		)
 		(pin "2"
 		)
@@
 		(in_bom yes)
 		(on_board yes)
-		(dnp no)
+		(dnp yes)
 		(property "Reference" "U11"
 			(at 147.32 81.1532 0)
@@
 		)
 		(property "Mouser Part Number" "926-LM386N-3/NOPB"
+			(at 137.16 76.2 0)
+			(effects
+				(font
+					(size 1.27 1.27)
+				)
+				(hide yes)
+			)
+		)
+		(property "LCSC" "DNF"
 			(at 137.16 76.2 0)
 			(effects
@@
 			)
 		)
-		(property "LCSC" "C49678"
+		(property "LCSC" "C113803"
 			(at 124.46 63.5 0)
 			(effects
@@
 			)
 		)
-		(property "LCSC" ""
+		(property "LCSC" "C1622"
 			(at 187.96 85.09 0)
 			(effects

Commit message: Auto stash before merge of "main" and "origin/main"
Parts:
- C56, LS1, R88, U11, VR1: now fitted
Changed lines of the file:
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@@
 		(in_bom yes)
 		(on_board yes)
-		(dnp yes)
+		(dnp no)
 		(fields_autoplaced yes)
 		(property "Reference" "C56"
@@
 		(in_bom yes)
 		(on_board yes)
-		(dnp yes)
+		(dnp no)
 		(property "Reference" "VR1"
 			(at 101.6 123.19 0)
@@
 		(in_bom yes)
 		(on_board yes)
-		(dnp yes)
+		(dnp no)
 		(property "Reference" "R88"
 			(at 53.6779 99.0388 90)
@@
 		(in_bom yes)
 		(on_board yes)
-		(dnp yes)
+		(dnp no)
 		(fields_autoplaced yes)
 		(property "Reference" "LS1"
@@
 		(in_bom yes)
 		(on_board yes)
-		(dnp yes)
+		(dnp no)
 		(property "Reference" "U11"
 			(at 147.32 81.1532 0)

Commit message: LED value change, added fix for FTDI power
Parts:
- R88: value 0R -> 47K
Changed lines of the file:
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@@
 			)
 		)
-		(property "Value" "0R"
+		(property "Value" "47K"
 			(at 55.9639 99.0388 90)
 			(effects
