File: Schematics/LT6502/LT6502.kicad_pcb (KiCad board)
At the start: 4 copper layers, 261 x 83 mm, 229 parts, among them IC1 ATF1508AS-7AX100, IC2 MP2636GR-P, IC3 W65C22S6TQG-14, J1 Conn_02x05_Odd_Even, J11 Conn_02x04_Odd_Even, J12 Conn_02x06_Odd_Even, J13 Conn_02x06_Odd_Even, J14 KeyConn, J15 Conn_01x06, J16 Conn_01x03, J18 Conn_01x03, J2 USBPD_PROG, J3 USB_C_Receptacle_USB2.0_16P, J4 BATTERY JST PH-2A, J5 Conn_02x20_Odd_Even, J6 USB_C_Receptacle_USB2.0_16P, J7 Conn_01x02, J8 Conn_02x26_Top_Bottom, J9 DIN41612_02x32_AC, Q1 STL9P3LLH6, Q2 IRLML6402, Q3 STL9P3LLH6, U1 TC1232, U10 FT245RNL, U11 LM386, U12 W65C51NxP, U2 W65C02S6TQG-14, U3 IS62C256AL, U4 IS62C256AL, U5 SST39SF010, U6 STUSB4500QTR, U7 AP63203WU, U8 TXS0108, U9 TXS0108, X1 28.322MHz, X2 1.8432MHz, Y1 ECS-P55-28.000MHZ-AN

Commit message: LED value change, added fix for FTDI power
Parts:
- R64: value 1K -> 4K7
- R84: value 1K -> 6K8
- R88: value 0R -> 47K
Changed lines of the file:
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@@
 			)
 		)
-		(property "Value" "1K"
+		(property "Value" "4K7"
 			(at 0 1.17 0)
 			(layer "F.Fab")
@@
 			)
 		)
-		(property "LCSC" "C11702"
+		(property "LCSC" ""
 			(at 0 0 0)
 			(unlocked yes)
@@
 			)
 		)
-		(property "Value" "0R"
+		(property "Value" "47K"
 			(at 0 1.17 0)
 			(layer "F.Fab")
@@
 			)
 		)
-		(property "Value" "1K"
+		(property "Value" "6K8"
 			(at 0 1.17 0)
 			(layer "F.Fab")
@@
 			)
 		)
-		(property "LCSC" "C11702"
+		(property "LCSC" ""
 			(at 0 0 0)
 			(unlocked yes)
@@
 		)
 	)
-	(gr_text_box "V1.0-V1.1 Changes\nAdded cutout for reset switch\nAdded cutout for LS1 and moved it\nExpanded pads on L2 for ease of soldering\nChange R46 to 51K\nChange R47 to 120K\nAdded Pull ups to SLOW0 and SLOW1\nAdd Display Data Enable line\nNote CF_nCS and CF_nRES are swapped (oops), fixed in CPLD\nCLK and CLK/2 are swapped in CPLD\nFixed battery connector polarity to save swapping wires.\nChange top of R57 from 5V to VSYS to stop odd charging behaviour"
+	(gr_text_box "V1.0-V1.1 Changes\nAdded cutout for reset switch\nAdded cutout for LS1 and moved it\nExpanded pads on L2 for ease of soldering\nChange R46 to 51K\nChange R47 to 120K\nAdded Pull ups to SLOW0 and SLOW1\nAdd Display Data Enable line\nNote CF_nCS and CF_nRES are swapped (oops), fixed in CPLD\nCLK and CLK/2 are swapped in CPLD\nFixed battery connector polarity to save swapping wires.\nChange top of R57 from 5V to VSYS to stop odd charging behaviour\nChange R64 and R84 to reduce LED brightness\nChange R88 to reduce distortion on speaker\n"
 		(start 265.4 178.5)
 		(end 338.3 210.9)
