File: Schematics/LT6502/LT6502.kicad_pcb (KiCad board)
At the start: 4 copper layers, 261 x 83 mm, 229 parts, among them IC1 ATF1508AS-7AX100, IC2 MP2636GR-P, IC3 W65C22S6TQG-14, J1 Conn_02x05_Odd_Even, J11 Conn_02x04_Odd_Even, J12 Conn_02x06_Odd_Even, J13 Conn_02x06_Odd_Even, J14 KeyConn, J15 Conn_01x06, J16 Conn_01x03, J18 Conn_01x03, J2 USBPD_PROG, J3 USB_C_Receptacle_USB2.0_16P, J4 BATTERY JST PH-2A, J5 Conn_02x20_Odd_Even, J6 USB_C_Receptacle_USB2.0_16P, J7 Conn_01x02, J8 Conn_02x26_Top_Bottom, J9 DIN41612_02x32_AC, Q1 STL9P3LLH6, Q2 IRLML6402, Q3 STL9P3LLH6, U1 TC1232, U10 FT245RNL, U11 LM386, U12 W65C51NxP, U2 W65C02S6TQG-14, U3 IS62C256AL, U4 IS62C256AL, U5 SST39SF010, U6 STUSB4500QTR, U7 AP63203WU, U8 TXS0108, U9 TXS0108, X1 28.322MHz, X2 1.8432MHz, Y1 ECS-P55-28.000MHZ-AN

Commit message: PCB/Schematic edits
moved speaker hole a little
made nRES resistor for display no fit (this upsets them for some reason)
Added diodes to ensure USB Console chip is powered when nothing attached (this causes issues with booting.
Parts:
- added D1: B5819W SL, Diode_SMD:D_SOD-123, F.Cu at (115.7, 127.8)
- added D14: B5819W SL, Diode_SMD:D_SOD-123, F.Cu at (121.0, 127.9)
Connections:
- FB1 pad 1: /60FAKE50/VUSB -> Net-(D1-A)
Routing:
- net /60FAKE50/VUSB: track 38.7 -> 41.7 mm
- net +5V: track 154.2 -> 156.9 mm, vias 58 -> 60
- net Net-(D1-A): track 0.00 -> 2.33 mm
Other:
- outline, holes or cut-outs redrawn
