File: Schematics/LT6502/Glue_Addr.kicad_sch (KiCad schematic)
At the start: 33 parts, among them IC1 ATF1508AS-7AX100, J1 Conn_02x05_Odd_Even, J15 Conn_01x06, J16 Conn_01x03, J18 Conn_01x03, X1 28.322MHz, Y1 ECS-P55-28.000MHZ-AN

Commit message: Updated Schematics
Added bulk capacitance with higher ESR to help with display PLL starting
Parts:
- removed Y1: ECS-P55-28.000MHZ-AN, Oscillator:Oscillator_SMD_EuroQuartz_XO53-4Pin_5.0x3.2mm, symbol Oscillator:ECS-2520MV-xxx-xx
- added R93, R94: 10k, Resistor_SMD:R_0402_1005Metric, symbol Device:R
- X1: value 28.322MHz -> 16MHz
Connections:
- net +5V: now also R93.2, R94.2
- net FT_nRXF: now also R93.1
- net FT_nTXE: now also R94.1
Other:
- moved on the sheet: R21, R22, R27
