File: Schematics/Multi-Ex/FPU.kicad_sch (KiCad schematic)
At the start: 16 parts, among them Q1 STL9P3LLH6, U1 MC68882_PLCC_68, U2 74HC245

Commit message: Multi-expansion card routed.
Parts:
- added R10, R11: 10K, Resistor_SMD:R_0402_1005Metric, symbol Device:R
Connections:
- net FPU_5V: now also R10.1, R11.1
- net FPU_nDSACK0: now also R10.2
- net FPU_nDSACK1: now also R11.2
