File: Schematics/Multi-Ex/Glue.kicad_sch (KiCad schematic)
At the start: 24 parts, among them IC2 ATF1508AS-7AX100, J16 Conn_01x03, J2 Conn_01x03, J4 Conn_02x05_Odd_Even, J5 Conn_01x03

Commit message: Multi-expansion card routed.
Connections:
- net RDY: now reaches IC2.92 (I/O_66)
Changed lines of the file:
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@@
+	(wire
+		(pts
+			(xy 62.23 95.25) (xy 77.47 95.25)
+		)
+		(stroke
+			(width 0)
+			(type default)
+		)
+	)
 	(wire
 		(pts
@@
 		)
 	)
+	(hierarchical_label "RDY"
+		(shape output)
+		(at 62.23 95.25 180)
+		(effects
+			(font
+				(size 1.27 1.27)
+			)
+			(justify right)
+		)
+	)
